File: 01 Hardware - developement/08 All_togother/08 All_togother.kicad_pcb (KiCad board)
At the start: 2 copper layers, 220.1 x 371.5 mm, 113 parts, among them IC2 STM32H7A3RIT6TR, J1 POLOLU-2593, J10 Conn_01x03_Pin, J11 Conn_01x03_Pin, J13 ftdi232, J15 ST-link cn3, J16 Boot, J2 ST-link cn6, J3 Conn_01x02_Pin, J4 Conn_01x02_Pin, J5 Conn_01x02_Pin, J6 Conn_01x03_Pin, J7 Conn_01x01_Socket, J8 Conn_01x02_Pin, J9 Conn_01x02_Pin, Q1 BC807, Q2 BC807, SW1 SW_Push_Dual, U1 24C16, U2 LM7805_TO220, X1 8.0MHz 20pF

Commit message: stm32 -hw- pull-up resistors 10k
Parts:
- R17, R18, R6, R7: value 4k7 -> 10k
Changed lines of the file:
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@@
   (net 99 "unconnected-(B7-----Pad4)")
   (net 100 "unconnected-(B7-----Pad8)")
-  (net 101 "unconnected-(B7-I2S_MLCK-PadI2S_4)")
+  (net 101 "unconnected-(B7-n{slash}c-PadI2S_4)")
   (net 102 "Net-(Q1-B)")
   (net 103 "Net-(Q2-B)")
@@
       (net 51 "/I2S_WS_esp32") (pinfunction "I2S_LRCLK") (pintype "input"))
     (pad "I2S_4" thru_hole oval (at -54.356 21.48) (size 1.7 1.7) (drill 1) (layers "*.Cu" "*.Mask")
-      (net 101 "unconnected-(B7-I2S_MLCK-PadI2S_4)") (pinfunction "I2S_MLCK") (pintype "input+no_connect"))
+      (net 101 "unconnected-(B7-n{slash}c-PadI2S_4)") (pinfunction "n/c") (pintype "no_connect"))
     (pad "I2S_5" thru_hole oval (at -54.356 24.02) (size 1.7 1.7) (drill 1) (layers "*.Cu" "*.Mask")
       (net 30 "/~{PS_Sust_ESP32}") (pinfunction "~{PS_Sust_ESP32}") (pintype "input"))
@@
     (property "Sheetfile" "08 All_togother.kicad_sch")
     (property "Sheetname" "")
-    (property "TME no." "SMD0603-4K7-1%")
+    (property "TME no." "RC0603FR-1310KL")
     (property "ki_description" "Resistor")
     (property "ki_keywords" "R res resistor")
@@
         (effects (font (size 1 1) (thickness 0.15)) (justify mirror))
     )
-    (fp_text value "4k7" (at 0 -1.43) (layer "B.Fab")
+    (fp_text value "10k" (at 0 -1.43) (layer "B.Fab")
         (effects (font (size 1 1) (thickness 0.15)) (justify mirror))
     )
@@
     (property "Sheetfile" "08 All_togother.kicad_sch")
     (property "Sheetname" "")
-    (property "TME no." "SMD0603-4K7-1%")
+    (property "TME no." "RC0603FR-1310KL")
     (property "ki_description" "Resistor")
     (property "ki_keywords" "R res resistor")
@@
         (effects (font (size 1 1) (thickness 0.15)) (justify mirror))
     )
-    (fp_text value "4k7" (at 0 -1.43) (layer "B.Fab")
+    (fp_text value "10k" (at 0 -1.43) (layer "B.Fab")
         (effects (font (size 1 1) (thickness 0.15)) (justify mirror))
     )
@@
     (property "Sheetfile" "08 All_togother.kicad_sch")
     (property "Sheetname" "")
-    (property "TME no." "SMD0603-4K7-1%")
+    (property "TME no." "RC0603FR-1310KL")
     (property "ki_description" "Resistor")
     (property "ki_keywords" "R res resistor")
@@
         (effects (font (size 1 1) (thickness 0.15)) (justify mirror))
     )
-    (fp_text value "4k7" (at 0 -1.43) (layer "B.Fab")
+    (fp_text value "10k" (at 0 -1.43) (layer "B.Fab")
         (effects (font (size 1 1) (thickness 0.15)) (justify mirror))
     )
@@
     (property "Sheetfile" "08 All_togother.kicad_sch")
     (property "Sheetname" "")
-    (property "TME no." "SMD0603-4K7-1%")
+    (property "TME no." "RC0603FR-1310KL")
     (property "ki_description" "Resistor")
     (property "ki_keywords" "R res resistor")
@@
         (effects (font (size 1 1) (thickness 0.15)) (justify mirror))
     )
-    (fp_text value "4k7" (at 0 -1.43) (layer "B.Fab")
+    (fp_text value "10k" (at 0 -1.43) (layer "B.Fab")
         (effects (font (size 1 1) (thickness 0.15)) (justify mirror))
     )

Commit message: all toogothert -hw- poprawiono crystal
Parts:
- C10, C11: value 30pF -> 30pF n.a.
Changed lines of the file:
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@@
     (property "Sheetname" "")
     (property "TME no." "C0603C300J5GAC")
+    (property "dnp" "")
     (property "ki_description" "Unpolarized capacitor")
     (property "ki_keywords" "cap capacitor")
@@
         (effects (font (size 1 1) (thickness 0.15)) (justify mirror))
     )
-    (fp_text value "30pF" (at 0 -1.43 90) (layer "B.Fab")
+    (fp_text value "30pF n.a." (at 0 -1.43 90) (layer "B.Fab")
         (effects (font (size 1 1) (thickness 0.15)) (justify mirror))
     )
@@
     (property "Sheetname" "")
     (property "TME no." "C0603C300J5GAC")
+    (property "dnp" "")
     (property "ki_description" "Unpolarized capacitor")
     (property "ki_keywords" "cap capacitor")
@@
         (effects (font (size 1 1) (thickness 0.15)) (justify mirror))
     )
-    (fp_text value "30pF" (at 0 -1.43 90) (layer "B.Fab")
-        (effects (font (size 1 1) (thickness 0.15)) (justify mirror))
-    )
+    (fp_text value "30pF n.a." (at 0 -1.43 90) (layer "B.Fab")
+        (effects (font (size 1 1) (thickness 0.15)) (justify mirror))
+    )
