File: 01 Hardware - developement/03b ESP32 bluetooth & HMI/esp32 bluetooth.kicad_sch (KiCad schematic)
At the start: 48 parts, among them J1 I2C, J2 UART, J3 power supply, J4 Jtag, J5 I2S, J8 Conn_01x01_Pin, SW10 Strapping button, SW8 Strapping button, SW9 Strapping button, U2 ESP32-DevKitC, U3 MCP23008

Commit message: ESP32 - porządek w firmware (tylko VS CODE) i na PCB )dodano złącza ESP PROG)
Parts:
- added D10, D11, D12, D5, D6, D7, D8, D9: ESD5Z3.3T1G, Diode_SMD:D_SOD-523, symbol Diode:ESD9B3.3ST5G
- added ESP-Prog1: Conn_02x03_Odd_Even, Connector_IDC:IDC-Header_2x03_P2.54mm_Vertical, symbol Connector_Generic:Conn_02x03_Odd_Even
- added J10, J11: Conn_01x02_Pin, Connector_PinHeader_1.27mm:PinHeader_1x02_P1.27mm_Vertical, symbol Connector:Conn_01x02_Pin
- added J9: Conn_02x05_Odd_Even, Connector_IDC:IDC-Header_2x05_P2.54mm_Vertical, symbol Connector_Generic:Conn_02x05_Odd_Even
Connections:
- net +3V3: now also J10.1 (Pin_1), J11.2 (Pin_2)
- net BT_UATR_RX: now also D6.1 (A1), ESP-Prog1.5 (Pin_5)
- net BT_UATR_TX: now also D7.1 (A1), ESP-Prog1.3 (Pin_3)
- net Debug_TCK: now also D11.1 (A1), J9.4 (Pin_4)
- net Debug_TDI: now also D9.1 (A1), J9.8 (Pin_8)
- net Debug_TDO: now also D10.1 (A1), J9.6 (Pin_6)
- net Debug_TMS: now also D12.1 (A1), J9.2 (Pin_2)
- net GNDD: now also D10.2 (A2), D11.2 (A2), D12.2 (A2), D5.2 (A2), D6.2 (A2), D7.2 (A2), D8.2 (A2), D9.2 (A2), ESP-Prog1.4 (Pin_4), J9.3 (Pin_3), J9.5 (Pin_5), J9.7 (Pin_7), J9.9 (Pin_9)
- new net: J11.1 (Pin_1), J9.1 (Pin_1)
- new net: ESP-Prog1.2 (Pin_2), J10.2 (Pin_2)
- new net ESP_EN: D8.1 (A1), ESP-Prog1.1 (Pin_1)
- new net ESP_IO0: D5.1 (A1), ESP-Prog1.6 (Pin_6)
- no-connect marks 17 -> 18
Other:
- note added: "W wersji finalnej wykasować jTag JLinka"
- note removed: "ERROR: Rezystor R57 powinien być podpięty to 3V3, bo podpięce do GND wprowadza ESP32 w stan programowania. Trzeba zienić to i w programie sterującyn ~{INT_request}."
- moved on the sheet: C1, C14, C15, D1, D2, D3, D4, J1, J2, J3, J4, J5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

Commit message: Do poprwy jest schemat rotary encodera
Other:
- note added: "TRZEBA POPRAWIĆ schematy rotary encodera!!! Styki sa podłączone niezgodnie z nota katalogową (chodzi o obszar 10kOhm)"
Changed lines of the file:
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@@
+		)
+	)
+	(text "TRZEBA POPRAWIĆ schematy rotary encodera!!!\nStyki sa podłączone niezgodnie z nota katalogową\n(chodzi o obszar 10kOhm)"
+		(exclude_from_sim no)
+		(at 262.382 27.178 0)
+		(effects
+			(font
+				(size 5.08 5.08)
+				(thickness 0.254)
+				(bold yes)
+				(color 255 2 43 1)
+			)
+			(justify left bottom)
+			(href "#2")
 		)
 	)
