File: 01 Hardware - developement/03b ESP32 bluetooth & HMI/esp32 bluetooth.kicad_sch (KiCad schematic)
At the start: 60 parts, among them J1 I2C, J10 Conn_01x02_Pin, J11 Conn_01x02_Pin, J2 UART, J3 power supply, J4 Jtag, J5 I2S, J8 Conn_01x01_Pin, J9 Conn_02x05_Odd_Even, SW10 Strapping button, SW8 Strapping button, SW9 Strapping button, U2 ESP32-DevKitC, U3 MCP23008

Commit message: poprawka esp32 GPIO0 z pulldown do pullup
Connections:
- net +3V3: now also R57.2
- net GNDD: no longer R57.2
Changed lines of the file:
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@@
+	(symbol
+		(lib_id "power:+3V3")
+		(at 101.6 109.22 0)
+		(unit 1)
+		(exclude_from_sim no)
+		(in_bom yes)
+		(on_board yes)
+		(dnp no)
+		(property "Reference" "#PWR071"
+			(at 101.6 113.03 0)
+			(effects
+				(font
+					(size 1.27 1.27)
+				)
+				(hide yes)
+			)
+		)
+		(property "Value" "+3V3"
+			(at 101.6001 105.41 90)
+			(effects
+				(font
+					(size 1.27 1.27)
+				)
+				(justify left)
+			)
+		)
+		(property "Footprint" ""
+			(at 101.6 109.22 0)
+			(effects
+				(font
+					(size 1.27 1.27)
+				)
+				(hide yes)
+			)
+		)
+		(property "Datasheet" ""
+			(at 101.6 109.22 0)
+			(effects
+				(font
+					(size 1.27 1.27)
+				)
+				(hide yes)
+			)
+		)
+		(property "Description" ""
+			(at 101.6 109.22 0)
+			(effects
+				(font
+					(size 1.27 1.27)
+				)
+			)
+		)
+		(pin "1"
+		)
+		(instances
+			(project "esp32 bluetooth"
+				(path "/85fd60db-6313-4d29-84e5-9ad356eb710e"
+					(reference "#PWR071")
+					(unit 1)
+				)
+			)
+		)
+	)
 	(symbol
 		(lib_id "power:+3V3")
@@
 					(unit 1)
 				)
-			)
-		)
-	)
-	(symbol
-		(lib_id "power:GNDD")
-		(at 101.6 109.22 180)
-		(unit 1)
-		(exclude_from_sim no)
-		(in_bom yes)
-		(on_board yes)
-		(dnp no)
-		(property "Reference" "#PWR071"
-			(at 101.6 102.87 0)
-			(effects
-				(font
-					(size 1.27 1.27)
-				)
-				(hide yes)
-			)
-		)
-		(property "Value" "GNDD"
-			(at 101.4984 105.283 0)
-			(effects
-				(font
-					(size 1.27 1.27)
-				)
-			)
-		)
-		(property "Footprint" ""
-			(at 101.6 109.22 0)
-			(effects
-				(font
-					(size 1.27 1.27)
-				)
-				(hide yes)
-			)
-		)
-		(property "Datasheet" ""
-			(at 101.6 109.22 0)
-			(effects
-				(font
-					(size 1.27 1.27)
-				)
-				(hide yes)
-			)
-		)
-		(property "Description" ""
-			(at 101.6 109.22 0)
-			(effects
-				(font
-					(size 1.27 1.27)
-				)
-			)
-		)
-		(pin "1"
-		)
-		(instances
-			(project "esp32 bluetooth"
-				(path "/85fd60db-6313-4d29-84e5-9ad356eb710e"
-					(reference "#PWR071")
-					(unit 1)
-				)
